Commit message: Added collision geometry to the URDF

File: puma560_description/urdf/puma560_robot.urdf (robot description, URDF)
Before this commit: robot Puma560, 7 links, 6 joints
Links:
- link link1: geometry collision mesh filename=../meshes/puma_link1.stl scale=0.0254 0.0254 0.0254; visual mesh filename=../meshes/puma_link1.stl scale=0.0254 0.0254 0.0254
- link link2: geometry collision mesh filename=../meshes/puma_link2.stl scale=0.0254 0.0254 0.0254; visual mesh filename=../meshes/puma_link2.stl scale=0.0254 0.0254 0.0254
- link link3: geometry collision mesh filename=../meshes/puma_link3.stl scale=0.0254 0.0254 0.0254; visual mesh filename=../meshes/puma_link3.stl scale=0.0254 0.0254 0.0254
- link link4: geometry collision mesh filename=../meshes/puma_link4.stl scale=0.0254 0.0254 0.0254; visual mesh filename=../meshes/puma_link4.stl scale=0.0254 0.0254 0.0254
- link link5: geometry collision mesh filename=../meshes/puma_link5.stl scale=0.0254 0.0254 0.0254; visual mesh filename=../meshes/puma_link5.stl scale=0.0254 0.0254 0.0254
- link link6: geometry collision mesh filename=../meshes/puma_link6.stl scale=0.0254 0.0254 0.0254; visual mesh filename=../meshes/puma_link6.stl scale=0.0254 0.0254 0.0254
- link link7: geometry collision mesh filename=../meshes/puma_link7.stl scale=0.0254 0.0254 0.0254; visual mesh filename=../meshes/puma_link7.stl scale=0.0254 0.0254 0.0254
